File: gbczero/gbczero.kicad_pcb (KiCad board)
At the start: 2 copper layers, 71.4 x 128 mm, 74 parts, among them J1 USB_B_Micro, J2 Conn_01x18, J4 AudioJack3_Switch, Q1 MMUN2133LT1G, Q2 PN2222A, Q3 PN2222A, Q4 AO3400A, SW1 SW_SPDT, SW2 SW_Push, U1 RASPBERRY_PI_ZERO_2_W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

Commit message: almost done
Parts:
- J4: footprint Connector_Audio:Jack_3.5mm_CUI_SJ1-3523N_Horizontal -> Connector_Audio:Jack_3.5mm_CUI_SJ1-3525N_Horizontal
- U5: moved to F.Cu
- moved U5 56.9 mm to (123.0, 139.2), turned to 0 degrees
- moved R13 12.1 mm to (120.0, 83.7), turned to -90 degrees
- moved R16 6.71 mm to (121.5, 71.5), turned to 180 degrees
- moved R26 4.26 mm to (165.5, 134.0)
- moved R27 2.92 mm to (169.0, 134.0)
- moved C14 2.05 mm to (121.0, 143.5)
- moved R24 1.72 mm to (120.5, 69.5), turned to 180 degrees
- moved C10 1.00 mm to (116.5, 146.8)
- moved C11 1.00 mm to (116.5, 150.7)
- moved U2 1.00 mm to (122.8, 150.6)
- moved L1 0.86 mm to (121.8, 50.2)
- moved LS1 0.40 mm to (174.9, 134.5)
- moved SW1 0.28 mm to (173.7, 63.3)
- moved Q1 0.11 mm to (133.8, 56.1)
- turned Q4 to 180 degrees
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Connections:
- R11 pad 1: Net-(U5-SDA) -> /FG_SDA
- R12 pad 1: Net-(U5-SCL) -> /FG_SCL
- U5 pad 7: Net-(U5-SCL) -> /FG_SCL
- U5 pad 8: Net-(U5-SDA) -> /FG_SDA
Routing:
- net GND: track 0.00 -> 374.6 mm, vias 1 -> 32
- net /VBAT: track 0.00 -> 323.3 mm, vias 0 -> 2
- net +3.3V: track 0.00 -> 302.6 mm, vias 0 -> 12
- net /DAC_LRCK: track 0.00 -> 172.3 mm
- net +5V: track 0.00 -> 145.7 mm, vias 0 -> 7
- net Net-(D4-K): track 0.00 -> 137.9 mm
- net /DAC_DIN: track 0.00 -> 137.6 mm
- net /FG_SCL: track 0.00 -> 126.8 mm
- net Net-(U4-THERM): track 0.00 -> 126.2 mm
- net /BTN_SEL: track 0.00 -> 124.5 mm
- net /FG_SDA: track 0.00 -> 119.5 mm
- net /PWR_HIGH: track 0.00 -> 116.9 mm, vias 0 -> 1
- net /CHARGING: track 0.00 -> 115.8 mm, vias 0 -> 3
- net /DAC_BCK: track 0.00 -> 113.1 mm
- net /PWR_EN: track 0.00 -> 112.5 mm
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- added copper zone on B.Cu, net GND
- added copper zone on F.Cu, net GND
Other:
- outline, holes or cut-outs redrawn

Commit message: zero errors
Parts:
- removed Q3: PN2222A, Package_TO_SOT_THT:TO-92_Inline
- added Q5: MMBT2222A, Package_TO_SOT_SMD:SOT-23, F.Cu at (115.9, 60.2)
- Q2: value PN2222A -> MMBT2222A; footprint Package_TO_SOT_THT:TO-92_Inline -> Package_TO_SOT_SMD:SOT-23
- moved Q2 5.30 mm to (115.7, 66.0)
Connections:
- Q2 pad 1: GND -> Net-(Q2-B)
- Q2 pad 2: Net-(Q2-B) -> GND
- R21 pad 2: Net-(Q2-C) -> Net-(Q5-C)
- R22 pad 2: Net-(Q2-B) -> Net-(Q5-B)
- R23 pad 2: Net-(Q3-C) -> Net-(Q2-C)
- R24 pad 2: Net-(Q3-B) -> Net-(Q2-B)
Routing:
- net GND: track 374.6 -> 384.2 mm, vias 32 -> 34
- net Net-(Q5-B): track 0.00 -> 7.50 mm
- net Net-(Q3-B): track 6.42 -> 0.00 mm
- net Net-(Q5-C): track 0.00 -> 5.91 mm
- net Net-(Q3-C): track 5.79 -> 0.00 mm
- net Net-(Q2-B): track 5.58 -> 7.93 mm
- net /LOW_BATTERY: track 91.0 -> 93.0 mm
- net /VBAT: track 323.3 -> 324.9 mm
- net /CHARGING_DIRECT: track 35.1 -> 35.9 mm
- net Net-(Q2-C): track 6.35 -> 5.79 mm

Commit message: Finished (maybe)
Parts:
- removed SW1: SW_SPDT, Button_Switch_SMD:SW_SPDT_PCM12
- added C16: 10uF, Capacitor_SMD:C_0603_1608Metric, B.Cu at (164.2, 123.5)
- added C17: 1uF, Capacitor_SMD:C_0603_1608Metric, B.Cu at (164.2, 125.5)
- added C18: 0.1uF, Capacitor_SMD:C_0603_1608Metric, B.Cu at (165.5, 131.0)
- added C19: 0.1uF, Capacitor_SMD:C_0603_1608Metric, B.Cu at (162.0, 134.8)
- added SW3: SW, Library:SW-SMD_4P-P1.50_L3.6-W11.3, B.Cu at (172.0, 64.8)
- C10: footprint Capacitor_SMD:C_0603_1608Metric -> Capacitor_Tantalum_SMD:CP_EIA-3216-18_Kemet-A
- C4: footprint Capacitor_SMD:C_0603_1608Metric -> Capacitor_Tantalum_SMD:CP_EIA-7343-31_Kemet-D
- L1: value 6.8uF -> 6.8uH
- SW2: footprint Button_Switch_SMD:SW_Push_1TS009xxxx-xxxx-xxxx_6x6x5mm -> Button_Switch_SMD:SW_Push_1P1T_XKB_TS-1187A
- moved C4 18.7 mm to (130.6, 68.2)
- moved C10 15.0 mm to (120.0, 132.2), turned to 0 degrees
- moved SW2 1.88 mm to (145.4, 135.1)
- moved R26 0.35 mm to (165.8, 134.2)
Connections:
- U3 pad 3: /AMP_INP -> Net-(U3-IN+)
- U3 pad 4: GND -> Net-(U3-IN-)
Routing:
- net +3.3V: track 302.6 -> 316.5 mm
- net Net-(U3-IN+): track 0.00 -> 13.6 mm
- net /AMP_INP: track 13.6 -> 6.40 mm
- net +5V: track 145.7 -> 152.4 mm, vias 7 -> 8
- net /VBAT: track 324.9 -> 329.1 mm
- net GND: track 384.2 -> 387.6 mm, vias 34 -> 36
- net Net-(U3-IN-): track 0.00 -> 2.27 mm
- net Net-(U4-THERM): track 126.2 -> 128.0 mm
- net /PWR_EN: track 112.5 -> 111.0 mm
- net Net-(U3-OUT-): track 23.7 -> 22.7 mm
- net /DAC_BCK: track 113.1 -> 112.2 mm
- net Net-(C9-Pad2): track 27.1 -> 28.0 mm
- net /DAC_DIN: track 137.6 -> 136.8 mm
- net /DAC_LRCK: track 172.3 -> 171.7 mm
