File: gbczero/gbczero.kicad_pcb (KiCad board)
At the start: 2 copper layers, 71.4 x 128 mm, 78 parts, among them J1 USB_B_Micro, J2 Conn_01x18, J4 AudioJack3_Switch, Q1 MMUN2133LT1G, Q2 MMBT2222A, Q4 AO3400A, Q5 MMBT2222A, SW2 SW_Push, SW3 SW, U1 RASPBERRY_PI_ZERO_2_W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

Commit message: Update
Parts:
- C18, C19: value 0.1uF -> 100nF
- C3, C7: value 4.7µF -> 4.7uF
- C4: value 220µF -> 220uF
- C5: value 10µF -> 10uF
- C6: value 2.2µF -> 2.2uF
Changed lines of the file:
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@@
 			)
 		)
-		(property "Value" "0.1uF"
+		(property "Value" "100nF"
 			(at 0 -1.43 0)
 			(layer "B.Fab")
@@
 			)
 		)
-		(property "Value" "0.1uF"
+		(property "Value" "100nF"
 			(at 0 -1.43 90)
 			(layer "B.Fab")
@@
 			)
 		)
-		(property "Value" "220µF"
+		(property "Value" "220uF"
 			(at 0 -3.1 0)
 			(layer "B.Fab")
@@
 			)
 		)
-		(property "Datasheet" ""
+		(property "Datasheet" "~"
 			(at 0 0 0)
 			(layer "B.Fab")
@@
 			)
 		)
-		(property "Description" ""
+		(property "Description" "Polarized capacitor"
 			(at 0 0 0)
 			(layer "B.Fab")
@@
 			)
 		)
-		(property "Value" "4.7µF"
+		(property "Value" "4.7uF"
 			(at 0 -1.43 0)
 			(layer "B.Fab")
@@
 			)
 		)
-		(property "Value" "2.2µF"
+		(property "Value" "2.2uF"
 			(at 0 -1.43 0)
 			(layer "B.Fab")
@@
 			)
 		)
-		(property "Value" "4.7µF"
+		(property "Value" "4.7uF"
 			(at 0 -1.43 0)
 			(layer "B.Fab")
@@
 			)
 		)
-		(property "Value" "10µF"
+		(property "Value" "10uF"
 			(at 0 -1.43 0)
 			(layer "B.Fab")
@@
 			)
 		)
-		(property "Datasheet" ""
+		(property "Datasheet" "~"
 			(at 0 0 180)
 			(layer "B.Fab")
@@
 			)
 		)
-		(property "Description" ""
+		(property "Description" "Polarized capacitor"
 			(at 0 0 180)
 			(layer "B.Fab")
@@
 		(sheetname "/")
 		(sheetfile "gbczero.kicad_sch")
-		(attr through_hole exclude_from_pos_files)
+		(attr through_hole)
 		(fp_line
 			(start 6 7.7)
@@
 			)
 		)
-		(property "Datasheet" ""
+		(property "Datasheet" "~"
 			(at 0 0 0)
 			(unlocked yes)
@@
 			)
 		)
-		(property "Description" ""
+		(property "Description" "Push button switch, generic, two pins"
 			(at 0 0 0)
 			(unlocked yes)
