File: gbczero/gbczero.kicad_sch (KiCad schematic)
At the start: 77 parts, among them J1 USB_B_Micro, J2 Conn_01x18, J4 AudioJack3_Switch, Q1 MMUN2133LT1G, Q2 PN2222A, Q3 PN2222A, Q4 AO3400A, SW1 SW_SPDT, SW2 SW_Push, U1 RASPBERRY_PI_ZERO_2_W, U11 74HC04, U12 74HC04, U2 PCM5102A, U3 PAM8302AAD, U4 MCP73833T-AMI_MF, U5 MAX17048G_T10, U6 74HC04, U7 TPS61030, U8 74HC00, U9 74HC10

Commit message: a
Parts:
- removed 4.7µF1: C, symbol Device:C
- removed 6.8µF1: L, symbol Device:L
- removed D5: LED_RGBA, symbol Device:LED_RGBA
- removed R14, R15: 2K, symbol Device:R
- removed U11, U12: 74HC04, symbol 74xx:74HC04
- added C15: 4.7uF, Capacitor_SMD:C_0603_1608Metric, symbol Device:C
- added D2: BAT54C, Package_TO_SOT_SMD:SOT-23, symbol Diode:BAT54C
- added L1: 6.8uF, Inductor_SMD:L_6.3x6.3_H3, symbol Device:L
- added R28: 1K, Resistor_SMD:R_0603_1608Metric, symbol Device:R
- added unit 3 of U6
- added unit 7 of U6
- added unit 5 of U8
- added unit 4 of U9
- BT1: footprint (none) -> Connector_JST:JST_PH_S2B-PH-K_1x02_P2.00mm_Horizontal
- BUTTON_A1, BUTTON_B1, DPAD_DOWN1, DPAD_LEFT1, DPAD_RIGHT1, DPAD_UP1: footprint (none) -> Library:GameBoy-DMG-BTN
- BUTTON_SELECT1, BUTTON_START1: footprint (none) -> Library:GameBoy-DMG-START-SEL
- C1, C10, C11, C12, C13, C14, C2, C3, C4, C5, C6, C7, C8, C9: footprint (none) -> Capacitor_SMD:C_0603_1608Metric
- D1: footprint (none) -> LED_THT:LED_D5.0mm-4_RGB
- J1: footprint (none) -> Connector_USB:USB_Micro-B_Molex_47346-0001
- J2: footprint (none) -> Connector_FFC-FPC:Hirose_FH12-18S-0.5SH_1x18-1MP_P0.50mm_Horizontal
- J4: footprint (none) -> Connector_Audio:Jack_3.5mm_CUI_SJ1-3523N_Horizontal
- LS1: footprint (none) -> Connector_PinHeader_2.54mm:PinHeader_1x02_P2.54mm_Vertical
- R1, R10, R11, R12, R13, R16, R17, R18, R19, R2, R20, R21, R22, R23, R24, R25, R26, R27, R3, R4, R5, R6, R7, R8, R9, TH1: footprint (none) -> Resistor_SMD:R_0603_1608Metric
- SW1: footprint (none) -> Button_Switch_SMD:SW_SPDT_PCM12
- SW2: footprint (none) -> Button_Switch_SMD:SW_Push_1TS009xxxx-xxxx-xxxx_6x6x5mm
- U4: footprint MCP73833T-AMI_MF:SON50P300X300X100-11N -> MCP73833T-AMI-MF:SON50P300X300X100-11N
- U6, U8, U9: footprint (none) -> Package_SO:SOIC-14_3.9x8.7mm_P1.27mm
Connections:
- net BTN_BOTTOM is gone; now on net DPAD_BOTTOM: DPAD_LEFT1.1 (A)
- net BTN_LEFT is gone; now on net DPAD_LEFT: DPAD_RIGHT1.1 (A)
- net +3.3V: now also D2.2, U6.14 (VCC), U8.14 (VCC), U9.14 (VCC); no longer D1.4 (A)
- net CHARGING: now also U8.4, U9.1, R28.1; no longer U6.1
- net GND: now also C15.2, L1.2, U6.7 (GND), U8.7 (GND), U9.7 (GND)
- net PWR_HIGH: now also U1.8 (GPIO14/TXD0)
- net PWR_OFF_HOTKEY: now also U1.33 (GPIO13)
- net VBAT: now reaches BT1.1 (+), C5.2, C7.2, C8.1, C9.1, R4.1, SW1.1 (A), U4.10 (VBAT), U4.9 (VBAT), U5.2 (CELL), U5.3 (VDD), U7.6 (VBAT), U7.8 (SYNC)
- net VBAT: now also C15.1, L1.1
- net at R22.1: now also U6.2
- net at U9.12: now also U6.5
- net FG_SDA: now reaches U1.3 (GPIO2/SDA1)
- net FG_SCL: now reaches U1.5 (GPIO3/SCL)
- net VBUS: now reaches C3.1, J1.1 (VBUS), U4.1 (VDD), U4.2 (VDD)
- net VBUS: now also D2.1
- net at R24.1: now also U6.6
- net at U8.6: now also U6.1
- net LED_GB renamed CHARGING_DIRECT
- net CHARGING_DIRECT: now also R28.2
- new net: D1.4 (A), D2.3
Other:
- moved on the sheet: BT1, BUTTON_A1, BUTTON_B1, BUTTON_SELECT1, BUTTON_START1, C1, C10, C11, C12, C13, C14, C2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

Commit message: almost done
Connections:
- net FG_SCL: now also R12.1, U5.7 (SCL)
- net FG_SDA: now also R11.1, U5.8 (SDA)
Changed lines of the file:
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@@
 	)
 	(junction
+		(at 341.63 116.84)
+		(diameter 0)
+		(color 0 0 0 0)
+	)
+	(junction
 		(at 289.56 106.68)
 		(diameter 0)
@@
 	)
 	(junction
+		(at 341.63 121.92)
+		(diameter 0)
+		(color 0 0 0 0)
+	)
+	(junction
 		(at 247.65 135.89)
 		(diameter 0)
@@
 	(wire
 		(pts
-			(xy 391.16 116.84) (xy 336.55 116.84)
+			(xy 336.55 116.84) (xy 341.63 116.84)
 		)
 		(stroke
@@
 	(wire
 		(pts
+			(xy 341.63 113.03) (xy 344.17 113.03)
+		)
+		(stroke
+			(width 0)
+			(type default)
+		)
+	)
+	(wire
+		(pts
 			(xy 198.12 139.7) (xy 198.12 140.97)
 		)
@@
 	(wire
 		(pts
+			(xy 341.63 121.92) (xy 381 121.92)
+		)
+		(stroke
+			(width 0)
+			(type default)
+		)
+	)
+	(wire
+		(pts
 			(xy 46.99 212.09) (xy 46.99 219.71)
 		)
@@
 	(wire
 		(pts
-			(xy 21.59 212.09) (xy 33.02 212.09)
+			(xy 341.63 125.73) (xy 344.17 125.73)
 		)
 		(stroke
@@
 	(wire
 		(pts
-			(xy 153.67 91.44) (xy 163.83 91.44)
+			(xy 21.59 212.09) (xy 33.02 212.09)
 		)
 		(stroke
@@
 	(wire
 		(pts
-			(xy 299.72 153.67) (xy 300.99 153.67)
+			(xy 153.67 91.44) (xy 163.83 91.44)
 		)
 		(stroke
@@
 	(wire
 		(pts
-			(xy 336.55 43.18) (xy 340.36 43.18)
+			(xy 299.72 153.67) (xy 300.99 153.67)
 		)
 		(stroke
@@
 	(wire
 		(pts
-			(xy 191.77 128.27) (xy 191.77 135.89)
+			(xy 336.55 43.18) (xy 340.36 43.18)
 		)
 		(stroke
@@
 	(wire
 		(pts
-			(xy 365.76 60.96) (xy 368.3 60.96)
+			(xy 191.77 128.27) (xy 191.77 135.89)
 		)
 		(stroke
@@
 	(wire
 		(pts
-			(xy 336.55 121.92) (xy 381 121.92)
+			(xy 365.76 60.96) (xy 368.3 60.96)
 		)
 		(stroke
@@
 	(wire
 		(pts
+			(xy 341.63 116.84) (xy 341.63 113.03)
+		)
+		(stroke
+			(width 0)
+			(type default)
+		)
+	)
+	(wire
+		(pts
 			(xy 190.5 43.18) (xy 199.39 43.18)
 		)
@@
 	(wire
 		(pts
+			(xy 341.63 116.84) (xy 391.16 116.84)
+		)
+		(stroke
+			(width 0)
+			(type default)
+		)
+	)
+	(wire
+		(pts
 			(xy 242.57 130.81) (xy 242.57 109.22)
 		)
@@
 	(wire
 		(pts
+			(xy 336.55 121.92) (xy 341.63 121.92)
+		)
+		(stroke
+			(width 0)
+			(type default)
+		)
+	)
+	(wire
+		(pts
 			(xy 370.84 170.18) (xy 370.84 153.67)
 		)
@@
 	(wire
 		(pts
+			(xy 341.63 121.92) (xy 341.63 125.73)
+		)
+		(stroke
+			(width 0)
+			(type default)
+		)
+	)
+	(wire
+		(pts
 			(xy 336.55 114.3) (xy 336.55 92.71)
 		)
@@
 		)
 	)
+	(label "FG_SCL"
+		(at 344.17 113.03 0)
+		(effects
+			(font
+				(size 1.27 1.27)
+			)
+			(justify left bottom)
+		)
+	)
 	(label "DISPLAY_RESET"
 		(at 48.26 102.87 180)
@@
 		(effects
 			(font
+				(size 1.27 1.27)
+			)
+			(justify left bottom)
+		)
+	)
+	(label "FG_SDA"
+		(at 344.17 125.73 0)
+		(effects
+			(font

Commit message: zero errors
Parts:
- removed Q2, Q3: PN2222A, Package_TO_SOT_THT:TO-92_Inline, symbol Transistor_BJT:PN2222A
- added Q2, Q5: MMBT2222A, Package_TO_SOT_SMD:SOT-23, symbol Transistor_BJT:MMBT2222A
Connections:
- net GND: now also Q2.2 (E), Q5.2 (E)
- net at R22.2: now also Q5.1 (B)
- net at R24.2: now also Q2.1 (B)
- net at R23.2: now also Q2.3 (C)
- net at R21.2: now also Q5.3 (C)
Changed lines of the file:
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@@
 	)
 	(symbol
-		(lib_id "Transistor_BJT:PN2222A")
-		(at 68.58 184.15 0)
-		(mirror y)
-		(unit 1)
-		(exclude_from_sim no)
-		(in_bom yes)
-		(on_board yes)
-		(dnp no)
-		(property "Reference" "Q3"
-			(at 63.5 182.8799 0)
-			(effects
-				(font
-					(size 1.27 1.27)
-				)
-				(justify left)
-			)
-		)
-		(property "Value" "PN2222A"
-			(at 63.5 185.4199 0)
-			(effects
-				(font
-					(size 1.27 1.27)
-				)
-				(justify left)
-			)
-		)
-		(property "Footprint" "Package_TO_SOT_THT:TO-92_Inline"
-			(at 63.5 186.055 0)
-			(effects
-				(font
-					(size 1.27 1.27)
-					(italic yes)
-				)
-				(justify left)
-				(hide yes)
-			)
-		)
-		(property "Datasheet" "https://www.onsemi.com/pub/Collateral/PN2222-D.PDF"
-			(at 68.58 184.15 0)
-			(effects
-				(font
-					(size 1.27 1.27)
-				)
-				(justify left)
-				(hide yes)
-			)
-		)
-		(property "Description" "1A Ic, 40V Vce, NPN Transistor, General Purpose Transistor, TO-92"
-			(at 68.58 184.15 0)
-			(effects
-				(font
-					(size 1.27 1.27)
-				)
-				(hide yes)
-			)
-		)
-		(pin "1"
-		)
-		(pin "2"
-		)
-		(pin "3"
-		)
-		(instances
-			(project "gbczero"
-				(path "/cfcfd9fa-fc73-4ab0-afa2-1bf19858b96d"
-					(reference "Q3")
-					(unit 1)
-				)
-			)
-		)
-	)
-	(symbol
 		(lib_id "Amplifier_Audio:PAM8302AAD")
 		(at 154.94 41.91 0)
@@
 	)
 	(symbol
+		(lib_id "Transistor_BJT:MMBT2222A")
+		(at 101.6 196.85 0)
+		(mirror y)
+		(unit 1)
+		(exclude_from_sim no)
+		(in_bom yes)
+		(on_board yes)
+		(dnp no)
+		(property "Reference" "Q5"
+			(at 96.52 195.5799 0)
+			(effects
+				(font
+					(size 1.27 1.27)
+				)
+				(justify left)
+			)
+		)
+		(property "Value" "MMBT2222A"
+			(at 96.52 198.1199 0)
+			(effects
+				(font
+					(size 1.27 1.27)
+				)
+				(justify left)
+			)
+		)
+		(property "Footprint" "Package_TO_SOT_SMD:SOT-23"
+			(at 96.52 198.755 0)
+			(effects
+				(font
+					(size 1.27 1.27)
+					(italic yes)
+				)
+				(justify left)
+				(hide yes)
+			)
+		)
+		(property "Datasheet" "https://assets.nexperia.com/documents/data-sheet/MMBT2222A.pdf"
+			(at 101.6 196.85 0)
+			(effects
+				(font
+					(size 1.27 1.27)
+				)
+				(justify left)
+				(hide yes)
+			)
+		)
+		(property "Description" "600mA Ic, 40V Vce, NPN Transistor, SOT-23"
+			(at 101.6 196.85 0)
+			(effects
+				(font
+					(size 1.27 1.27)
+				)
+				(hide yes)
+			)
+		)
+		(pin "2"
+		)
+		(pin "1"
+		)
+		(pin "3"
+		)
+		(instances
+			(project ""
+				(path "/cfcfd9fa-fc73-4ab0-afa2-1bf19858b96d"
+					(reference "Q5")
+					(unit 1)
+				)
+			)
+		)
+	)
+	(symbol
 		(lib_id "power:GND")
 		(at 309.88 43.18 270)
@@
 	)
 	(symbol
+		(lib_id "Transistor_BJT:MMBT2222A")
+		(at 68.58 184.15 0)
+		(mirror y)
+		(unit 1)
+		(exclude_from_sim no)
+		(in_bom yes)
+		(on_board yes)
+		(dnp no)
+		(property "Reference" "Q2"
+			(at 63.5 182.8799 0)
+			(effects
+				(font
+					(size 1.27 1.27)
+				)
+				(justify left)
+			)
+		)
+		(property "Value" "MMBT2222A"
+			(at 63.5 185.4199 0)
+			(effects
+				(font
+					(size 1.27 1.27)
+				)
+				(justify left)
+			)
+		)
+		(property "Footprint" "Package_TO_SOT_SMD:SOT-23"
+			(at 63.5 186.055 0)
+			(effects
+				(font
+					(size 1.27 1.27)
+					(italic yes)
+				)
+				(justify left)
+				(hide yes)
+			)
+		)
+		(property "Datasheet" "https://assets.nexperia.com/documents/data-sheet/MMBT2222A.pdf"
+			(at 68.58 184.15 0)
+			(effects
+				(font
+					(size 1.27 1.27)
+				)
+				(justify left)
+				(hide yes)
+			)
+		)
+		(property "Description" "600mA Ic, 40V Vce, NPN Transistor, SOT-23"
+			(at 68.58 184.15 0)
+			(effects
+				(font
+					(size 1.27 1.27)
+				)
+				(hide yes)
+			)
+		)
+		(pin "2"
+		)
+		(pin "1"
+		)
+		(pin "3"
+		)
+		(instances
+			(project "gbczero"
+				(path "/cfcfd9fa-fc73-4ab0-afa2-1bf19858b96d"
+					(reference "Q2")
+					(unit 1)
+				)
+			)
+		)
+	)
+	(symbol
 		(lib_id "Device:R")
 		(at 332.74 40.64 90)
@@
 					(unit 1)
 				)
-			)
-		)
-	)
-	(symbol
-		(lib_id "Transistor_BJT:PN2222A")
-		(at 101.6 196.85 0)
-		(mirror y)
-		(unit 1)
-		(exclude_from_sim no)
-		(in_bom yes)
-		(on_board yes)
-		(dnp no)
-		(property "Reference" "Q2"
-			(at 96.52 195.5799 0)
-			(effects
-				(font
-					(size 1.27 1.27)
-				)
-				(justify left)
-			)
-		)
-		(property "Value" "PN2222A"
-			(at 96.52 198.1199 0)
-			(effects
-				(font
-					(size 1.27 1.27)
-				)
-				(justify left)
-			)
-		)
-		(property "Footprint" "Package_TO_SOT_THT:TO-92_Inline"
-			(at 96.52 198.755 0)
-			(effects
-				(font
-					(size 1.27 1.27)
-					(italic yes)
-				)
-				(justify left)
-				(hide yes)
-			)
-		)
-		(property "Datasheet" "https://www.onsemi.com/pub/Collateral/PN2222-D.PDF"
-			(at 101.6 196.85 0)
-			(effects
-				(font
-					(size 1.27 1.27)
-				)
-				(justify left)
-				(hide yes)
-			)
-		)
-		(property "Description" "1A Ic, 40V Vce, NPN Transistor, General Purpose Transistor, TO-92"
-			(at 101.6 196.85 0)
-			(effects
-				(font
-					(size 1.27 1.27)
-				)
-				(hide yes)
-			)
-		)
-		(pin "1"
-		)
-		(pin "2"
-		)
-		(pin "3"
-		)
-		(instances
-			(project ""
-				(path "/cfcfd9fa-fc73-4ab0-afa2-1bf19858b96d"
-					(reference "Q2")
-					(unit 1)
-				)

Commit message: Finished (maybe)
Parts:
- removed SW1: SW_SPDT, Button_Switch_SMD:SW_SPDT_PCM12, symbol Switch:SW_SPDT
- added C16: 10uF, Capacitor_SMD:C_0603_1608Metric, symbol Device:C
- added C17: 1uF, Capacitor_SMD:C_0603_1608Metric, symbol Device:C
- added C18, C19: 0.1uF, Capacitor_SMD:C_0603_1608Metric, symbol Device:C
- added SW3: SW, Library:SW-SMD_4P-P1.50_L3.6-W11.3, symbol New_Library:SK-1391L-2
- C10: footprint Capacitor_SMD:C_0603_1608Metric -> Capacitor_Tantalum_SMD:CP_EIA-3216-18_Kemet-A; symbol Device:C -> Device:C_Polarized
- C4: footprint Capacitor_SMD:C_0603_1608Metric -> Capacitor_Tantalum_SMD:CP_EIA-7343-31_Kemet-D; symbol Device:C -> Device:C_Polarized
- L1: value 6.8uF -> 6.8uH
- SW2: footprint Button_Switch_SMD:SW_Push_1TS009xxxx-xxxx-xxxx_6x6x5mm -> Button_Switch_SMD:SW_Push_1P1T_XKB_TS-1187A
Connections:
- net +5V: now also C16.1, C17.1
- net AMP_INP: now also C19.1; no longer U3.3 (IN+)
- net GND: now also C16.2, C17.2, C18.1; no longer U3.4 (IN-)
- net VBAT: now also SW3.4
- net at C9.2, D4.1 (A), R18.2: now also SW3.1, SW3.2
- new net: C19.2, U3.3 (IN+)
- new net: C18.2, U3.4 (IN-)
- no-connect marks 1 -> 18
Other:
- moved on the sheet: C9

Commit message: Update
Parts:
- C18, C19: value 0.1uF -> 100nF
- C3, C7: value 4.7µF -> 4.7uF
- C4: value 220µF -> 220uF
- C5: value 10µF -> 10uF
- C6: value 2.2µF -> 2.2uF
Changed lines of the file:
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@@
 			)
 		)
-		(property "Value" "10µF"
+		(property "Value" "10uF"
 			(at 295.91 160.02 90)
 			(effects
@@
 			)
 		)
-		(property "Value" "4.7µF"
+		(property "Value" "4.7uF"
 			(at 363.22 167.6399 0)
 			(effects
@@
 			)
 		)
-		(property "Value" "0.1uF"
+		(property "Value" "100nF"
 			(at 165.354 36.576 0)
 			(effects
@@
 			)
 		)
-		(property "Value" "4.7µF"
+		(property "Value" "4.7uF"
 			(at 295.91 148.59 90)
 			(effects
@@
 			)
 		)
-		(property "Value" "220µF"
+		(property "Value" "220uF"
 			(at 190.5 146.0499 0)
 			(effects
@@
 			)
 		)
-		(property "Value" "0.1uF"
+		(property "Value" "100nF"
 			(at 171.45 39.116 0)
 			(effects
@@
 			)
 		)
-		(property "Value" "2.2µF"
+		(property "Value" "2.2uF"
 			(at 187.96 140.9699 0)
 			(effects

Commit message: I'll change some things in a bit
Parts:
- added J3: USB_B_Micro, Connector_USB:USB_Micro-B_Molex_47346-0001, symbol Connector:USB_B_Micro
- added U10: USBLC6-2SC6, Package_TO_SOT_SMD:SOT-23-6, symbol Power_Protection:USBLC6-2SC6
Connections:
- net +5V: now also J3.1 (VBUS), U10.5 (VBUS)
- net GND: now also J3.5 (GND), J3.6 (Shield), U10.2 (GND)
- new net: J3.2 (D-), U10.3 (I/O2)
- new net: J3.3 (D+), U10.1 (I/O1)
- new net DATA_NEG: U10.4 (I/O2)
- new net DATA_POS: U10.6 (I/O1)
- no-connect marks 18 -> 19
